File: hardware/cocktail-machine/cocktail-machine.sch (KiCad schematic (older format))
At the start: 12 parts

Commit message: Finalize schematic
Parts:
- added J? (x2): Barrel_Jack, symbol Connector:Barrel_Jack
- added Q? (x2): IRF5305, symbol Device:Q_PMOS_GDS
- added U?: LM2596_Buck, symbol ulib_Modules:LM2596_Buck
- M?: value Motor_Servo -> MG996R
- R?: value 100 -> 100R
- R?: value 27/1/2W -> 27R/1|2W
- gave numbers to parts that had none: 1
Connections:
- net +5V: now also U?.3 (OUT+); no longer A?.5 (+5V)
- net GND: now also J?.2, Q?.1 (G), U?.2 (IN-), U?.4 (OUT-)
- net VCC renamed +7.5V
- net +7.5V: now also Q?.3 (S), U?.1 (IN+)
- new net: J?.1, Q?.2 (D) (x2)
- new net +12V: Q?.3 (S)
- new net GNDREF: J?.2, Q?.1 (G)
- no-connect marks 15 -> 16
Other:
- note added: "+12VDC SUPPLY"
- note added: "+5VDC SUPPLY"
- note added: "IR TRANSMITTER/RECEIVER"
- note added: "POWER FLAGS"
- note added: "POWER SUPPLY"
- moved on the sheet: A?, C?, D?, DS?, M?, Q?, R?, U?

Commit message: Reroute Arduino Uno's pins on schematic
Connections:
- net IR_RX: now also A?.16 (D1/TX); no longer A?.19 (D4)
- net IR_TX: now also A?.17 (D2); no longer A?.20 (D5)
- net MISO: no longer DS?.13 (T_DO)
- net MOSI: no longer DS?.12 (T_DIN)
- net MOTOR_PWM: now also A?.15 (D0/RX); no longer A?.18 (D3)
- net SCK: no longer DS?.10 (T_CLK)
- net T_IRQ: now also A?.18 (D3); no longer A?.21 (D6)
- net T_~CS: now also A?.21 (D6); no longer A?.22 (D7)
- new net T_CLK: A?.22 (D7), DS?.10 (T_CLK)
- new net T_DIN: A?.20 (D5), DS?.12 (T_DIN)
- new net T_DO: A?.19 (D4), DS?.13 (T_DO)
- no-connect marks 16 -> 13
Changed lines of the file:
@@
 Wire Wire Line
 	5150 4450 5100 4450
-Text Label 5100 4450 2    50   ~ 0
+Text Label 5100 4150 2    50   ~ 0
 MOTOR_PWM
 NoConn ~ 5750 3750
@@
 T_IRQ
 Text Label 4800 1650 0    50   ~ 0
-MISO
+T_DO
 Text Label 4800 1750 0    50   ~ 0
-MOSI
+T_DIN
 Text Label 4800 1850 0    50   ~ 0
 T_~CS
 Text Label 4800 1950 0    50   ~ 0
-SCK
+T_CLK
 Wire Wire Line
 	5150 5250 5100 5250
@@
 Text Label 5100 5150 2    50   ~ 0
 LCD_~CS
-Text Label 5100 4750 2    50   ~ 0
-T_IRQ
-Text Label 5100 4850 2    50   ~ 0
-T_~CS
 Wire Wire Line
 	5100 4550 5150 4550
@@
 Text Label 6950 2600 2    50   ~ 0
 IR_TX
-Text Label 5100 4550 2    50   ~ 0
+Text Label 5100 4250 2    50   ~ 0
 IR_RX
-Text Label 5100 4650 2    50   ~ 0
+Text Label 5100 4350 2    50   ~ 0
 IR_TX
 NoConn ~ 6150 5450
 NoConn ~ 6150 5550
-NoConn ~ 5150 4350
-NoConn ~ 5150 4250
-NoConn ~ 5150 4150
 NoConn ~ 6150 4550
 NoConn ~ 6150 4350
@@
 Text Notes 6650 1300 0    50   ~ 0
 IR TRANSMITTER/RECEIVER
+Wire Wire Line
+	5150 4150 5100 4150
+Wire Wire Line
+	5150 4250 5100 4250
+Wire Wire Line
+	5150 4350 5100 4350
+Text Label 5100 4450 2    50   ~ 0
+T_IRQ
+Text Label 5100 4550 2    50   ~ 0
+T_DO
+Text Label 5100 4650 2    50   ~ 0
+T_DIN
+Text Label 5100 4750 2    50   ~ 0
+T_~CS
+Text Label 5100 4850 2    50   ~ 0
+T_CLK
 $EndSCHEMATC

Commit message: Reroute Arduino pins. Recalculate IRTX resistor values
Parts:
- added R?: 200R, symbol Device:R
- R?: value 27R/1|2W -> 30R/0.6W
- R?: value 6.2k -> 6.8k
Connections:
- net IR_TX: now also A?.20 (D5), R?.2; no longer A?.17 (D2), R?.2
- net MOTOR_PWM: now also A?.18 (D3); no longer A?.15 (D0/RX)
- net T_DIN: now also A?.15 (D0/RX); no longer A?.20 (D5)
- net T_IRQ: now also A?.17 (D2); no longer A?.18 (D3)
- new net: R?.1, R?.2
Changed lines of the file:
@@
 Sheet 1 2
 Title "Cocktail Machine"
-Date "2020-04-26"
+Date "2020-04-30"
 Rev "1"
 Comp "Pesho & Valka Inc."
@@
 	1    5650 4750
 	1    0    0    -1
-$EndComp
-$Comp
-L Device:LED D?
-U 1 1 5E943420
-P 7650 1800
-F 0 "D?" V 7700 1950 50  0000 C CNN
-F 1 "IR_LED" V 7600 2000 50  0000 C CNN
-F 2 "" H 7650 1800 50  0001 C CNN
-F 3 "~" H 7650 1800 50  0001 C CNN
-	1    7650 1800
-	0    -1   -1   0
 $EndComp
 $Comp
@@
 Wire Wire Line
 	7650 1950 7650 2050
-$Comp
-L Device:R R?
-U 1 1 5E9752B5
-P 7650 2200
-F 0 "R?" H 7720 2246 50  0000 L CNN
-F 1 "27R/1|2W" H 7720 2155 50  0000 L CNN
-F 2 "" V 7580 2200 50  0001 C CNN
-F 3 "~" H 7650 2200 50  0001 C CNN
-	1    7650 2200
-	1    0    0    -1
-$EndComp
 Wire Wire Line
 	7650 2350 7650 2400
@@
 Wire Wire Line
 	5150 4450 5100 4450
-Text Label 5100 4150 2    50   ~ 0
+Text Label 5100 4450 2    50   ~ 0
 MOTOR_PWM
 NoConn ~ 5750 3750
@@
 P 7150 2600
 F 0 "R?" V 6943 2600 50  0000 C CNN
-F 1 "6.2k" V 7034 2600 50  0000 C CNN
+F 1 "6.8k" V 7034 2600 50  0000 C CNN
 F 2 "" V 7080 2600 50  0001 C CNN
 F 3 "~" H 7150 2600 50  0001 C CNN
@@
 Wire Wire Line
 	7000 2600 6950 2600
-Text Label 6950 2600 2    50   ~ 0
+Text Label 6600 2600 2    50   ~ 0
 IR_TX
 Text Label 5100 4250 2    50   ~ 0
 IR_RX
-Text Label 5100 4350 2    50   ~ 0
+Text Label 5100 4650 2    50   ~ 0
 IR_TX
 NoConn ~ 6150 5450
@@
 NoConn ~ 6150 4150
 Wire Notes Line
-	6650 3150 10800 3150
-Wire Notes Line
 	10800 3150 10800 1300
-Wire Notes Line
-	10800 1300 6650 1300
-Wire Notes Line
-	6650 1300 6650 3150
 $Comp
 L Connector:Barrel_Jack J?
@@
 Wire Wire Line
 	5150 4350 5100 4350
-Text Label 5100 4450 2    50   ~ 0
+Text Label 5100 4350 2    50   ~ 0
 T_IRQ
 Text Label 5100 4550 2    50   ~ 0
 T_DO
-Text Label 5100 4650 2    50   ~ 0
+Text Label 5100 4150 2    50   ~ 0
 T_DIN
 Text Label 5100 4750 2    50   ~ 0
@@
 Text Label 5100 4850 2    50   ~ 0
 T_CLK
+$Comp
+L Device:R R?
+U 1 1 5EAD7C8F
+P 6800 2600
+F 0 "R?" V 6593 2600 50  0000 C CNN
+F 1 "200R" V 6684 2600 50  0000 C CNN
+F 2 "" V 6730 2600 50  0001 C CNN
+F 3 "~" H 6800 2600 50  0001 C CNN
+	1    6800 2600
+	0    1    1    0
+$EndComp
+Wire Wire Line
+	6650 2600 6600 2600
+Wire Notes Line
+	6300 1300 6300 3150
+Wire Notes Line
+	6300 3150 10800 3150
+Wire Notes Line
+	6300 1300 10800 1300
+$Comp
+L Device:LED D?
+U 1 1 5E943420
+P 7650 1800
+F 0 "D?" V 7700 1950 50  0000 C CNN
+F 1 "IR_LED" V 7600 2000 50  0000 C CNN
+F 2 "" H 7650 1800 50  0001 C CNN
+F 3 "~" H 7650 1800 50  0001 C CNN
+	1    7650 1800
+	0    -1   -1   0
+$EndComp
+$Comp
+L Device:R R?
+U 1 1 5E9752B5
+P 7650 2200
+F 0 "R?" H 7720 2246 50  0000 L CNN
+F 1 "30R/0.6W" H 7720 2155 50  0000 L CNN
+F 2 "" V 7580 2200 50  0001 C CNN
+F 3 "~" H 7650 2200 50  0001 C CNN
+	1    7650 2200
+	1    0    0    -1
+$EndComp
 $EndSCHEMATC
