File: hardware/cocktail-machine/valve-interface.sch (KiCad schematic (older format))
At the start: 13 parts

Commit message: Finalize schematic
Parts:
- gave numbers to parts that had none: 12

Commit message: Final schematic version
Parts:
- gave numbers to parts that had none: 1
Connections:
- net +12V: now also K1.NO1, K1.NO2, K1.NO3, K1.NO4, K1.NO5, K1.NO6; no longer K1.NC1, K1.NC2, K1.NC3, K1.NC4, K1.NC5, K1.NC6
Changed lines of the file:
@@
 	4300 6500 4300 6550
 $Comp
-L power:GND #PWR?
+L power:GND #PWR024
 U 1 1 5EB6054B
 P 4300 6550
-F 0 "#PWR?" H 4300 6300 50  0001 C CNN
+F 0 "#PWR024" H 4300 6300 50  0001 C CNN
 F 1 "GND" H 4305 6377 50  0000 C CNN
 F 2 "" H 4300 6550 50  0001 C CNN
@@
 	4300 1000 4300 950
 $Comp
-L power:+5V #PWR?
+L power:+5V #PWR023
 U 1 1 5EB60552
 P 4300 950
-F 0 "#PWR?" H 4300 800 50  0001 C CNN
+F 0 "#PWR023" H 4300 800 50  0001 C CNN
 F 1 "+5V" H 4315 1123 50  0000 C CNN
 F 2 "" H 4300 950 50  0001 C CNN
@@
 P 4300 3750
 AR Path="/5EB60560" Ref="K?"  Part="1"
-AR Path="/5EB4C628/5EB60560" Ref="K?"  Part="1"
-F 0 "K?" H 3950 6400 50  0000 C CNN
+AR Path="/5EB4C628/5EB60560" Ref="K1"  Part="1"
+F 0 "K1" H 3950 6400 50  0000 C CNN
 F 1 "Relay_Module_8" H 4650 6400 50  0000 C CNN
 F 2 "" V 4780 4145 50  0001 C CNN
@@
 NoConn ~ 4900 2125
 NoConn ~ 4900 2350
-NoConn ~ 4900 3000
 $Comp
 L Motor:Motor_DC M?
@@
 	5750 3650 5650 3650
 Connection ~ 5650 3650
-NoConn ~ 4900 3650
 $Comp
 L Motor:Motor_DC M?
@@
 	5150 3800 5150 4075
 Connection ~ 5650 4300
-NoConn ~ 4900 4300
 $Comp
 L Motor:Motor_DC M?
@@
 	5750 4950 5650 4950
 Connection ~ 5650 4950
-NoConn ~ 4900 4950
 $Comp
 L Motor:Motor_DC M?
@@
 	5750 5600 5650 5600
 Connection ~ 5650 5600
-NoConn ~ 4900 5600
 $Comp
 L Motor:Motor_DC M?
@@
 	5750 6250 5650 6250
 Connection ~ 5650 6250
-NoConn ~ 4900 6250
 Wire Wire Line
 	3700 1475 3550 1475
@@
 CTRL1
 $Comp
-L power:+12V #PWR?
-U 1 1 5EA76F21
-P 5050 2500
-F 0 "#PWR?" H 5050 2350 50  0001 C CNN
-F 1 "+12V" H 5065 2673 50  0000 C CNN
-F 2 "" H 5050 2500 50  0001 C CNN
-F 3 "" H 5050 2500 50  0001 C CNN
-	1    5050 2500
-	1    0    0    -1
-$EndComp
-Wire Wire Line
-	5050 2550 5050 2500
-Wire Wire Line
-	4900 2550 5050 2550
-$Comp
-L power:+12V #PWR?
-U 1 1 5EA7C293
-P 5050 3150
-F 0 "#PWR?" H 5050 3000 50  0001 C CNN
-F 1 "+12V" H 5065 3323 50  0000 C CNN
-F 2 "" H 5050 3150 50  0001 C CNN
-F 3 "" H 5050 3150 50  0001 C CNN
-	1    5050 3150
-	1    0    0    -1
-$EndComp
-Wire Wire Line
-	5050 3200 5050 3150
-Wire Wire Line
-	4900 3200 5050 3200
-$Comp
-L power:+12V #PWR?
-U 1 1 5EA81199
-P 5050 3800
-F 0 "#PWR?" H 5050 3650 50  0001 C CNN
-F 1 "+12V" H 5065 3973 50  0000 C CNN
-F 2 "" H 5050 3800 50  0001 C CNN
-F 3 "" H 5050 3800 50  0001 C CNN
-	1    5050 3800
-	1    0    0    -1
-$EndComp
-Wire Wire Line
-	5050 3850 5050 3800
-Wire Wire Line
-	4900 3850 5050 3850
-$Comp
-L power:+12V #PWR?
-U 1 1 5EA85DA8
-P 5050 4450
-F 0 "#PWR?" H 5050 4300 50  0001 C CNN
-F 1 "+12V" H 5065 4623 50  0000 C CNN
-F 2 "" H 5050 4450 50  0001 C CNN
-F 3 "" H 5050 4450 50  0001 C CNN
-	1    5050 4450
-	1    0    0    -1
-$EndComp
-Wire Wire Line
-	5050 4500 5050 4450
-Wire Wire Line
-	4900 4500 5050 4500
-$Comp
-L power:+12V #PWR?
-U 1 1 5EA8ADE5
-P 5050 5100
-F 0 "#PWR?" H 5050 4950 50  0001 C CNN
-F 1 "+12V" H 5065 5273 50  0000 C CNN
-F 2 "" H 5050 5100 50  0001 C CNN
-F 3 "" H 5050 5100 50  0001 C CNN
-	1    5050 5100
-	1    0    0    -1
-$EndComp
-Wire Wire Line
-	5050 5150 5050 5100
-Wire Wire Line
-	4900 5150 5050 5150
-$Comp
-L power:+12V #PWR?
-U 1 1 5EA8F6FF
-P 5050 5750
-F 0 "#PWR?" H 5050 5600 50  0001 C CNN
-F 1 "+12V" H 5065 5923 50  0000 C CNN
-F 2 "" H 5050 5750 50  0001 C CNN
-F 3 "" H 5050 5750 50  0001 C CNN
-	1    5050 5750
-	1    0    0    -1
-$EndComp
-Wire Wire Line
-	5050 5800 5050 5750
-Wire Wire Line
-	4900 5800 5050 5800
-$Comp
-L power:GNDREF #PWR?
+L power:GNDREF #PWR031
 U 1 1 5EA9CAFF
 P 5750 3000
-F 0 "#PWR?" H 5750 2750 50  0001 C CNN
+F 0 "#PWR031" H 5750 2750 50  0001 C CNN
 F 1 "GNDREF" V 5755 2872 50  0000 R CNN
 F 2 "" H 5750 3000 50  0001 C CNN
@@
 $EndComp
 $Comp
-L power:GNDREF #PWR?
+L power:GNDREF #PWR032
 U 1 1 5EA9D3B3
 P 5750 3650
-F 0 "#PWR?" H 5750 3400 50  0001 C CNN
+F 0 "#PWR032" H 5750 3400 50  0001 C CNN
 F 1 "GNDREF" V 5755 3522 50  0000 R CNN
 F 2 "" H 5750 3650 50  0001 C CNN
@@
 	5750 4300 5650 4300
 $Comp
-L power:GNDREF #PWR?
+L power:GNDREF #PWR033
 U 1 1 5EA9E79F
 P 5750 4300
-F 0 "#PWR?" H 5750 4050 50  0001 C CNN
+F 0 "#PWR033" H 5750 4050 50  0001 C CNN
 F 1 "GNDREF" V 5755 4172 50  0000 R CNN
 F 2 "" H 5750 4300 50  0001 C CNN
@@
 $EndComp
 $Comp
-L power:GNDREF #PWR?
+L power:GNDREF #PWR034
 U 1 1 5EAAD59B
 P 5750 4950
-F 0 "#PWR?" H 5750 4700 50  0001 C CNN
+F 0 "#PWR034" H 5750 4700 50  0001 C CNN
 F 1 "GNDREF" V 5755 4822 50  0000 R CNN
 F 2 "" H 5750 4950 50  0001 C CNN
@@
 $EndComp
 $Comp
-L power:GNDREF #PWR?
+L power:GNDREF #PWR035
 U 1 1 5EAAE7B7
 P 5750 5600
-F 0 "#PWR?" H 5750 5350 50  0001 C CNN
+F 0 "#PWR035" H 5750 5350 50  0001 C CNN
 F 1 "GNDREF" V 5755 5472 50  0000 R CNN
 F 2 "" H 5750 5600 50  0001 C CNN
@@
 $EndComp
 $Comp
-L power:GNDREF #PWR?
+L power:GNDREF #PWR036
 U 1 1 5EAAFDFC
 P 5750 6250
-F 0 "#PWR?" H 5750 6000 50  0001 C CNN
+F 0 "#PWR036" H 5750 6000 50  0001 C CNN
 F 1 "GNDREF" V 5755 6122 50  0000 R CNN
 F 2 "" H 5750 6250 50  0001 C CNN
@@
 	0    -1   -1   0
 $EndComp
+$Comp
+L power:+12V #PWR025
+U 1 1 5ED51656
+P 4950 3000
+F 0 "#PWR025" H 4950 2850 50  0001 C CNN
+F 1 "+12V" V 4965 3128 50  0000 L CNN
+F 2 "" H 4950 3000 50  0001 C CNN
+F 3 "" H 4950 3000 50  0001 C CNN
+	1    4950 3000
+	0    1    1    0
+$EndComp
+Wire Wire Line
+	4900 3000 4950 3000
+NoConn ~ 4900 2550
+$Comp
+L power:+12V #PWR026
+U 1 1 5EDC3FB4
+P 4950 3650
+F 0 "#PWR026" H 4950 3500 50  0001 C CNN
+F 1 "+12V" V 4965 3778 50  0000 L CNN
+F 2 "" H 4950 3650 50  0001 C CNN
+F 3 "" H 4950 3650 50  0001 C CNN
+	1    4950 3650
+	0    1    1    0
+$EndComp
+Wire Wire Line
+	4950 3650 4900 3650
+NoConn ~ 4900 3200
+NoConn ~ 4900 3850
+Wire Wire Line
+	4900 4300 4950 4300
+$Comp
+L power:+12V #PWR027
+U 1 1 5EDCBFBC
+P 4950 4300
+F 0 "#PWR027" H 4950 4150 50  0001 C CNN
+F 1 "+12V" V 4965 4428 50  0000 L CNN
+F 2 "" H 4950 4300 50  0001 C CNN
+F 3 "" H 4950 4300 50  0001 C CNN
+	1    4950 4300
+	0    1    1    0
+$EndComp
+NoConn ~ 4900 4500
+$Comp
+L power:+12V #PWR028
+U 1 1 5EDCEC63
+P 4950 4950
+F 0 "#PWR028" H 4950 4800 50  0001 C CNN
+F 1 "+12V" V 4965 5078 50  0000 L CNN
+F 2 "" H 4950 4950 50  0001 C CNN
+F 3 "" H 4950 4950 50  0001 C CNN
+	1    4950 4950
+	0    1    1    0
+$EndComp
+Wire Wire Line
+	4950 4950 4900 4950
+NoConn ~ 4900 5150
+$Comp
+L power:+12V #PWR029
+U 1 1 5EDD2A3F
+P 4950 5600
+F 0 "#PWR029" H 4950 5450 50  0001 C CNN
+F 1 "+12V" V 4965 5728 50  0000 L CNN
+F 2 "" H 4950 5600 50  0001 C CNN
+F 3 "" H 4950 5600 50  0001 C CNN
+	1    4950 5600
+	0    1    1    0
+$EndComp
+Wire Wire Line
+	4950 5600 4900 5600
+NoConn ~ 4900 5800
+$Comp
+L power:+12V #PWR030
+U 1 1 5EDD9653
+P 4950 6250
+F 0 "#PWR030" H 4950 6100 50  0001 C CNN
+F 1 "+12V" V 4965 6378 50  0000 L CNN
+F 2 "" H 4950 6250 50  0001 C CNN
+F 3 "" H 4950 6250 50  0001 C CNN
+	1    4950 6250
+	0    1    1    0
+$EndComp
+Wire Wire Line
+	4950 6250 4900 6250
 $EndSCHEMATC
